File: project-nrf-garage-remote.kicad_pcb (KiCad board)
At the start: 2 copper layers, 34.5 x 27 mm, 9 parts, among them J1 Screw_Terminal_01x02, J2 Screw_Terminal_01x04, Q1 BSS138W, Q2 BSS138W

Commit message: Update pcb
Parts:
- added R2: PU, Resistor_SMD:R_0603_1608Metric, F.Cu at (38.5, 25.6)
- R1: value PD -> PU
- moved R1 7.90 mm to (38.5, 30.9), turned to 180 degrees
- moved Q1 2.10 mm to (38.5, 23.4)
- moved Q2 1.35 mm to (38.5, 28.6), turned to 0 degrees
Connections:
- J2 pad 1: /uc_send -> VDD
- J2 pad 2: /uc_recv -> /uc_send
- J2 pad 3: GND -> /uc_recv
- J2 pad 4: unconnected-(J2-Pin_4-Pad4) -> GND
- Q1 pad 1: /uc_send -> VDD
- Q1 pad 2: GND -> /uc_send
- Q2 pad 1: /motor_data -> VDD
- Q2 pad 2: GND -> /uc_recv
- Q2 pad 3: /uc_recv -> /motor_data
- R1 pad 1: /uc_send -> VDD
- R1 pad 2: GND -> /uc_recv
Routing:
- net VDD: track 0.00 -> 17.8 mm
- net GND: track 9.22 -> 6.60 mm, vias 5 -> 2
Other:
- board text added: "François Gervais 17 oct. 2024 v2.0.0"
- board text added: "Vdd"
- board text removed: "-"
- board text removed: "François Gervais 15 oct. 2024 v1.0.0"
